File: CAO_TrackPulse/CAO_TrackPulse.kicad_sch (KiCad schematic)
At the start: 0 parts

Commit message: Intialisation_Fixer
Parts:
- added U1: STM32L431CBTx, Package_QFP:LQFP-48_7x7mm_P0.5mm, symbol MCU_ST_STM32L4:STM32L431CBTx
Connections:
- new net: U1.23 (VSS), U1.35 (VSS), U1.47 (VSS)
Changed lines of the file:
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@@
 		(company "Arnaud & Augustin")
+	)
+	(symbol
+		(lib_id "MCU_ST_STM32L4:STM32L431CBTx")
+		(at 170.18 99.06 0)
+		(unit 1)
+		(body_style 1)
+		(exclude_from_sim no)
+		(in_bom yes)
+		(on_board yes)
+		(in_pos_files yes)
+		(dnp no)
+		(fields_autoplaced yes)
+		(property "Reference" "U1"
+			(at 174.8633 137.16 0)
+			(show_name no)
+			(do_not_autoplace no)
+			(effects
+				(font
+					(size 1.27 1.27)
+				)
+				(justify left)
+			)
+		)
+		(property "Value" "STM32L431CBTx"
+			(at 174.8633 139.7 0)
+			(show_name no)
+			(do_not_autoplace no)
+			(effects
+				(font
+					(size 1.27 1.27)
+				)
+				(justify left)
+			)
+		)
+		(property "Footprint" "Package_QFP:LQFP-48_7x7mm_P0.5mm"
+			(at 157.48 134.62 0)
+			(hide yes)
+			(show_name no)
+			(do_not_autoplace no)
+			(effects
+				(font
+					(size 1.27 1.27)
+				)
+				(justify right)
+			)
+		)
+		(property "Datasheet" "https://www.st.com/resource/en/datasheet/stm32l431cb.pdf"
+			(at 170.18 99.06 0)
+			(hide yes)
+			(show_name no)
+			(do_not_autoplace no)
+			(effects
+				(font
+					(size 1.27 1.27)
+				)
+			)
+		)
+		(property "Description" "STMicroelectronics Arm Cortex-M4 MCU, 128KB flash, 64KB RAM, 80 MHz, 1.71-3.6V, 38 GPIO, LQFP48"
+			(at 170.18 99.06 0)
+			(hide yes)
+			(show_name no)
+			(do_not_autoplace no)
+			(effects
+				(font
+					(size 1.27 1.27)
+				)
+			)
+		)
+		(pin "5"
+		)
+		(pin "18"
+		)
+		(pin "20"
+		)
+		(pin "22"
+		)
+		(pin "25"
+		)
+		(pin "29"
+		)
+		(pin "23"
+		)
+		(pin "13"
+		)
+		(pin "27"
+		)
+		(pin "26"
+		)
+		(pin "8"
+		)
+		(pin "3"
+		)
+		(pin "9"
+		)
+		(pin "4"
+		)
+		(pin "11"
+		)
+		(pin "1"
+		)
+		(pin "10"
+		)
+		(pin "12"
+		)
+		(pin "7"
+		)
+		(pin "6"
+		)
+		(pin "15"
+		)
+		(pin "16"
+		)
+		(pin "2"
+		)
+		(pin "14"
+		)
+		(pin "17"
+		)
+		(pin "19"
+		)
+		(pin "21"
+		)
+		(pin "24"
+		)
+		(pin "28"
+		)
+		(pin "40"
+		)
+		(pin "42"
+		)
+		(pin "33"
+		)
+		(pin "32"
+		)
+		(pin "38"
+		)
+		(pin "36"
+		)
+		(pin "37"
+		)
+		(pin "43"
+		)
+		(pin "31"
+		)
+		(pin "34"
+		)
+		(pin "39"
+		)
+		(pin "44"
+		)
+		(pin "35"
+		)
+		(pin "45"
+		)
+		(pin "30"
+		)
+		(pin "41"
+		)
+		(pin "46"
+		)
+		(pin "48"
+		)
+		(pin "47"
+		)
+		(instances
+			(project "CAO_TrackPulse"
+				(path "/7e0a8435-d431-4348-b986-f618cdfc0819"
+					(reference "U1")
+					(unit 1)
+				)
+			)
+		)
 	)
 	(sheet_instances

Commit message: Init_CAO
Parts:
- added J1: Conn_01x07_SIM7080G, symbol Connector:Conn_01x07_Socket
- added U2: W25Q64JVSSIQ, Package_SO:SOIC-8_5.3x5.3mm_P1.27mm, symbol Memory_Flash:W25Q32JVSS
- added U3: RN4871, RF_Module:Microchip_RN4871, symbol RF_Bluetooth:RN4871
- added U4: MCP73831-2-OT, Package_TO_SOT_SMD:SOT-23-5, symbol Battery_Management:MCP73831-2-OT
- added U5: TPS7A0533PDBV, Package_TO_SOT_SMD:SOT-23-5, symbol Regulator_Linear:TPS7A0533PDBV

Commit message: CAO_carte_principale_FINI
Parts:
- removed J1: Conn_01x07_SIM7080G, symbol Connector:Conn_01x07_Socket
- removed U1: STM32L431CBTx, Package_QFP:LQFP-48_7x7mm_P0.5mm, symbol MCU_ST_STM32L4:STM32L431CBTx
- removed U4: MCP73831-2-OT, Package_TO_SOT_SMD:SOT-23-5, symbol Battery_Management:MCP73831-2-OT
- added C1, C2: 4,7 µF, symbol Device:C
- added C10, C11, C12, C13, C14, C18, C19, C21, C4, C9: 100nF, symbol Device:C
- added C15, C16: 8,2pF, symbol Device:C
- added C17, C3, C8: 1µF, symbol Device:C
- added C20: 10µF, symbol Device:C_Polarized_Small
- added C5: 22µF, symbol Device:C
- added C6: 0,1µF, symbol Device:C
- added C7: 2,2µF, symbol Device:C
- added D1: LED, symbol Device:LED
- added D2: 1N4148W, Diode_SMD:D_SOD-123, symbol Diode:1N4148W
- added F1: Fuse, symbol Device:Fuse
- added J1: Conn_01x08_Screen_E_Peper, symbol Connector:Conn_01x08_Socket
- added J2: B2B-PH-K-S, B2B-PH-K-S:JST_B2B-PH-K-S, symbol B2B-PH-K-S:B2B-PH-K-S
- added J3: Conn_01x05_ADD, symbol Connector:Conn_01x05_Socket
- added J4: USB_C_Receptacle_USB2.0_16P, symbol Connector:USB_C_Receptacle_USB2.0_16P
- added J5: Conn_01x06_SWD, symbol Connector:Conn_01x06_Socket
- added LS1: CMT-8530S-SMT, CMT-8530S-SMT:CUI_CMT-8530S-SMT, symbol CMT-8530S-SMT:CMT-8530S-SMT
- added Q2: AO3400A, Package_TO_SOT_SMD:SOT-23, symbol Transistor_FET:AO3400A
- added R1, R2: 5,1 kΩ, symbol Device:R
- added R10, R12, R14, R15: 10k, symbol Device:R
- added R11, R13: 1M, symbol Device:R
- added R3: 100Ω, symbol Device:R
- added R4: 10KΩ, symbol Device:R
- added R5: 1k, symbol Device:R
- added R6: 2k, symbol Device:R
- added R7: 56k, symbol Device:R
- added R8: 300k, symbol Device:R
- added R9: 10K, symbol Device:R
- added SW1, SW2, SW3: CK_KMS2xxGP, Button_Switch_SMD:SW_SPST_CK_KMS2xxGP, symbol Switch:CK_KMS2xxGP
- added SW4: SW_DIP_x01, symbol Switch:SW_DIP_x01
- added U1: STM32L433CCTx, Package_QFP:LQFP-48_7x7mm_P0.5mm, symbol MCU_ST_STM32L4:STM32L433CCTx
- added U4: USBLC6-2SC6, Package_TO_SOT_SMD:SOT-23-6, symbol Power_Protection:USBLC6-2SC6
- added U7: LIS3DH, Package_LGA:LGA-16_3x3mm_P0.5mm_LayoutBorder3x5y, symbol Sensor_Motion:LIS3DH
- added U8: MCP73832-2-OT, Package_TO_SOT_SMD:SOT-23-5, symbol Battery_Management:MCP73832-2-OT
- added U9: TPS25200DRVR, TPS25200DRVR:SON65P200X200X80-7N, symbol TPS25200DRVR:TPS25200DRVR
- added Y1: 32.768 kHz, symbol Device:Crystal_GND24_Small
Connections:
- net QUADSPI_BK1_NCS: now reaches U2.1 (~{CS})
- net QUADSPI_BK1_NCS: now also R9.2, U1.12 (PA2)
- net QUADSPI_BK1_IO1: now reaches U2.2 (DO/IO_{1})
- net QUADSPI_BK1_IO1: now also U1.18 (PB0)
- net QUADSPI_BK1_IO2: now reaches U2.3 (~{WP}/IO_{2})
- net QUADSPI_BK1_IO2: now also U1.17 (PA7)
- net GND: now reaches U2.4 (GND)
- net GND: now also U3.13 (GND), U3.2 (GND), U5.2 (GND), C1.1, C10.2, C11.2, C12.2, C13.2, C14.1, C15.2, C16.1, C17.2, C18.1, C19.2, C2.2, C20.2, C21.2, C3.1, C4.1, C5.2, C6.1, C7.2, C8.1, C9.1, D1.1 (K), J1.7 (Pin_7), J2.2, J3.4 (Pin_4), J4.A1 (GND), J4.A12 (GND), J4.B1 (GND), J4.B12 (GND), J4.SH (SHIELD), J5.4 (Pin_4), Q2.2 (S), R1.2, R10.2, R13.2, R2.2, R4.2, R6.2, R7.2, SW1.1, SW2.1, SW3.1, U1.23 (VSS), U1.35 (VSS), U1.47 (VSS), U1.8 (VSSA), U4.2 (GND), U7.10 (GND), U7.12 (GND), U7.5 (GND), U7.7 (SDO), U8.2 (V_{SS}), U9.5 (GND), U9.7 (EXP), Y1.2 (G), Y1.4 (G)
- net QUADSPI_BK1_IO0: now reaches U2.5 (DI/IO_{0})
- net QUADSPI_BK1_IO0: now also U1.19 (PB1)
- net QUADSPI_CLK: now reaches U2.6 (CLK)
- net QUADSPI_CLK: now also U1.13 (PA3)
- net QUADSPI_BK1_IO3: now reaches U2.7 (~{HOLD}/~{RESET}/IO_{3})
- net QUADSPI_BK1_IO3: now also U1.16 (PA6)
- net +3V3: now reaches U2.8 (VCC)
- net +3V3: now also U3.14 (VBAT), U5.5 (OUT), C10.1, C11.1, C12.1, C13.1, C14.2, C17.1, C18.2, C19.1, C20.1, C7.1, C9.2, J1.8 (Pin_8), J5.3 (Pin_3), R12.1, R14.2, R15.2, R9.1, SW4.1, U1.1 (VBAT), U1.24 (VDD), U1.36 (VDDUSB), U1.48 (VDD), U1.9 (VDDA), U7.1 (VDD_IO), U7.14 (VDD), U7.8 (CS)
- net RST_BLE: now reaches U3.10 (RST)
- net RST_BLE: now also R12.2, U1.5 (PH0)
- net RTS_BLE: now reaches U3.11 (P0_0)
- net RTS_BLE: now also U1.25 (PB12)
- net TX_BLE: now reaches U3.7 (UART_RX)
- net TX_BLE: now also U1.22 (PB11)
- net RX_BLE: now reaches U3.8 (UART_TX)
- net RX_BLE: now also U1.21 (PB10)
- net CTS_BLE: now reaches U3.9 (P3_6)
- net CTS_BLE: now also U1.26 (PB13)
- net +BATT: now reaches U5.1 (IN)
- net +BATT: now also U5.3 (EN), C2.1, C8.2, D2.1 (K), F1.2, J3.5 (Pin_5), LS1.P, R11.2, U8.3 (V_{BAT})
- new net: Q2.1 (G), R3.1, R4.1
- new net: D1.2 (A), R5.1
- new net: C15.1, U1.4 (PC15), Y1.1
- new net: C16.2, U1.3 (PC14), Y1.3
- new net: D2.2 (A), LS1.N, Q2.3 (D)
- new net: R8.2, U9.4 (EN)
- new net: R10.1, SW4.2, U1.44 (PH3)
- new net: R7.1, U9.2 (ILIM)
- new net: F1.1, J2.1
- new net: R6.1, U8.5 (PROG)
- new net: J4.B5 (CC2), R2.1
- new net: J4.A7 (D-), J4.B7 (D-), U4.1 (I/O1)
- new net: J4.A6 (D+), J4.B6 (D+), U4.3 (I/O2)
- new net: J4.A5 (CC1), R1.1
- new net +5V: C1.2, C5.1, U8.4 (V_{DD}), U9.1 (OUT)
- new net ACC_INT1: U1.11 (PA1), U7.11 (INT1)
- new net ACC_SCL: R15.1, U1.45 (PB8), U7.4 (SPC)
- new net ACC_SDA: R14.1, U1.46 (PB9), U7.6 (SDI)
- new net BAT_SENSE: C21.1, R11.1, R13.1, U1.14 (PA4)
- new net BAT_STAT: U1.42 (PB6), U8.1 (STAT)
- new net BP1: SW1.2, U1.20 (PB2)
- new net BP2: SW2.2, U1.2 (PC13)
- new net BUZZER_PWM: R3.2, U1.10 (PA0)
- new net D+: U1.33 (PA12), U4.4 (I/O2)
- new net D-: U1.32 (PA11), U4.6 (I/O1)
- new net EPD_BUSY: J1.1 (Pin_1), U1.28 (PB15)
- new net EPD_CS: J1.4 (Pin_4), U1.6 (PH1)
- new net EPD_DC: J1.3 (Pin_3), U1.38 (PA15)
- new net EPD_MOSI: J1.5 (Pin_5), U1.41 (PB5)
- new net EPD_RST: J1.2 (Pin_2), U1.29 (PA8)
- new net EPD_SCK: J1.6 (Pin_6), U1.15 (PA5)
- new net FAULT: U1.43 (PB7), U9.3 (~{FAULT})
- new net LED1: R5.2, U1.40 (PB4)
- new net NRST: C4.2, J5.2 (Pin_2), SW3.2, U1.7 (NRST)
- new net PWRKEY: J3.3 (Pin_3), U1.27 (PB14)
- new net RX_SIM7080G: J3.2 (Pin_2), U1.31 (PA10)
- new net SWCLK: J5.5 (Pin_5), U1.37 (PA14)
- new net SWDIO: J5.6 (Pin_6), U1.34 (PA13)
- new net SWO: J5.1 (Pin_1), U1.39 (PB3)
- new net TX_SIM7080G: J3.1 (Pin_1), U1.30 (PA9)
- new net VBUS: C3.2, C6.2, J4.A4 (VBUS), J4.A9 (VBUS), J4.B4 (VBUS), J4.B9 (VBUS), R8.1, U4.5 (VBUS), U9.6 (IN)
- no-connect marks 0 -> 17
Other:
- moved on the sheet: U2, U3, U5
