File: CAO_TrackPulse/CAO_TrackPulse.kicad_sch (KiCad schematic)
At the start: 59 parts, among them J1 Conn_01x08_Screen_E_Peper, J2 B2B-PH-K-S, J3 Conn_01x05_ADD, J4 USB_C_Receptacle_USB2.0_16P, J5 Conn_01x06_SWD, Q2 AO3400A, SW1 CK_KMS2xxGP, SW2 CK_KMS2xxGP, SW3 CK_KMS2xxGP, SW4 SW_DIP_x01, U1 STM32L433CCTx, U2 W25Q64JVSSIQ, U3 RN4871, U4 USBLC6-2SC6, U5 TPS7A0533PDBV, U7 LIS3DH, U8 MCP73832-2-OT, U9 TPS25200DRVR, Y1 32.768 kHz

Commit message: Empreinte_assigne
Parts:
- removed C20: 10µF, symbol Device:C_Polarized_Small
- removed Y1: 32.768 kHz, symbol Device:Crystal_GND24_Small
- added C20: 10µF, Capacitor_SMD:C_0805_2012Metric_Pad1.18x1.45mm_HandSolder, symbol Device:C
- added J6: Conn_01x04_ADD_2, Connector_PinHeader_2.54mm:PinHeader_1x04_P2.54mm_Vertical, symbol Connector:Conn_01x04_Socket
- added Y1: Crystal, Crystal:Crystal_SMD_3215-2Pin_3.2x1.5mm, symbol Device:Crystal
- C1, C10, C11, C12, C13, C14, C17, C18, C19, C2, C21, C3, C4, C5, C6, C7, C8, C9, R1, R10, R11, R12, R13, R14, R15, R2, R3, R4, R5, R6, R7, R8, R9: footprint (none) -> Capacitor_SMD:C_0805_2012Metric_Pad1.18x1.45mm_HandSolder
- C15, C16: value 8,2pF -> 12pF; footprint (none) -> Capacitor_SMD:C_0805_2012Metric_Pad1.18x1.45mm_HandSolder
- D1: footprint (none) -> LED_SMD:LED_0805_2012Metric_Pad1.15x1.40mm_HandSolder
- F1: footprint (none) -> Fuse:Fuse_0805_2012Metric_Pad1.15x1.40mm_HandSolder
- J1: footprint (none) -> Connector_PinHeader_2.54mm:PinHeader_1x08_P2.54mm_Vertical
- J3: value Conn_01x05_ADD -> Conn_01x05_ADD_1; footprint (none) -> Connector_PinHeader_2.54mm:PinHeader_1x05_P2.54mm_Vertical
- J4: footprint (none) -> Connector_USB:USB_C_Receptacle_HRO_TYPE-C-31-M-12
- J5: footprint (none) -> Connector:Tag-Connect_TC2030-IDC-NL_2x03_P1.27mm_Vertical
- SW4: footprint (none) -> Button_Switch_SMD:SW_DIP_SPSTx01_Slide_Omron_A6S-110x_W8.9mm_P2.54mm
Connections:
- net +3V3: now also C20.1, J6.1 (Pin_1)
- net GND: now also C20.2, J6.2 (Pin_2)
- net at C15.1, U1.4 (PC15): now also Y1.1
- net at C16.2, U1.3 (PC14): now also Y1.2
- net SWO: no longer names the net of J5.1 (Pin_1)
- net SWO: no longer U1.39 (PB3)
- new net DTR_SIM7080G: J6.3 (Pin_3), U1.39 (PB3)
- no-connect marks 17 -> 19
Other:
- moved on the sheet: C15, C16, C21, J3, R11, R13

Commit message: rootage_main
Parts:
- LS1: footprint CMT-8530S-SMT:CUI_CMT-8530S-SMT -> buzzer:MagneticBuzzer_CUI_CMT-8504
- U9: footprint TPS25200DRVR:SON65P200X200X80-7N -> Package_SON:WSON-6-1EP_2x2mm_P0.65mm_EP1x1.6mm
Connections:
- net EPD_MOSI: now also J1.6 (Pin_6); no longer J1.5 (Pin_5)
- net EPD_SCK: now also J1.5 (Pin_5); no longer J1.6 (Pin_6)
Changed lines of the file:
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@@
 		)
 	)
-	(label "EPD_MOSI"
-		(at 156.21 33.02 0)
-		(effects
-			(font
-				(size 1.27 1.27)
-			)
-			(justify left bottom)
-		)
-	)
 	(label "ACC_SDA"
 		(at 138.43 252.73 0)
@@
 		)
 	)
+	(label "EPD_SCK"
+		(at 156.21 33.02 0)
+		(effects
+			(font
+				(size 1.27 1.27)
+			)
+			(justify left bottom)
+		)
+	)
 	(label "LED1"
 		(at 297.18 120.65 0)
@@
 		)
 	)
-	(label "EPD_SCK"
-		(at 156.21 30.48 0)
-		(effects
-			(font
-				(size 1.27 1.27)
-			)
-			(justify left bottom)
-		)
-	)
 	(label "QUADSPI_CLK"
 		(at 303.53 209.55 0)
@@
 		)
 	)
+	(label "EPD_MOSI"
+		(at 156.21 30.48 0)
+		(effects
+			(font
+				(size 1.27 1.27)
+			)
+			(justify left bottom)
+		)
+	)
 	(label "RST_BLE"
 		(at 297.18 90.17 0)
@@
 			)
 		)
-		(property "Footprint" "TPS25200DRVR:SON65P200X200X80-7N"
+		(property "Footprint" "Package_SON:WSON-6-1EP_2x2mm_P0.65mm_EP1x1.6mm"
 			(at 57.15 121.92 0)
 			(hide yes)
@@
 			)
 		)
-		(property "Footprint" "CMT-8530S-SMT:CUI_CMT-8530S-SMT"
+		(property "Footprint" "buzzer:MagneticBuzzer_CUI_CMT-8504"
 			(at 238.76 160.02 0)
 			(hide yes)
